File: ono-kairo/ono-kairo.kicad_sch (KiCad schematic)
At the start: 20 parts, among them J1 Conn_02x01, J2 Conn_02x02_Top_Bottom, U1 MCP3208, U2 DS18B20, U3 MCP6002-xMC

Commit message: Add files via upload
Parts:
- added CE0: CE0, MountingHole:MountingHole_2.2mm_M2_DIN965_Pad, symbol Mechanical:MountingHole_Pad
- added CLK1: CLK, MountingHole:MountingHole_2.2mm_M2_DIN965_Pad, symbol Mechanical:MountingHole_Pad
- added MISO1: MISO, MountingHole:MountingHole_2.2mm_M2_DIN965_Pad, symbol Mechanical:MountingHole_Pad
- added MOSI1: MOSI, MountingHole:MountingHole_2.2mm_M2_DIN965_Pad, symbol Mechanical:MountingHole_Pad
- J2: value Conn_02x02_Top_Bottom -> 02x02_Bottom
- renumbered R1 to 10k1, R7 to 10k2, R6 to 10k3, R2 to 1k1, H5 to 3.3V1, U2 to DS18B20, H4 to GND1, H3 to GPIO16, H2 to GPIO20, H1 to GPIO21
Connections:
- net CE0: no longer names the net of U1.10 (~{CS}/SHDN)
- net CE0: now also CE0.1
- net CLK: no longer names the net of U1.13 (CLK)
- net CLK: now also CLK1.1
- net MISO: no longer names the net of U1.12 (Dout)
- net MISO: now also MISO1.1
- net MOSI: no longer names the net of U1.11 (Din)
- net MOSI: now also MOSI1.1
